Commit message: 5.18门控

File: usv_ws/src/usv_description/urdf/wamv.urdf (robot description, URDF)
Before this commit: robot fog_usv, 5 links, 4 joints
Links:
- removed link radar_link
- added link als_lidar_link; visual cylinder length=0.12 radius=0.12
- added link gated_camera_link; visual box size=0.20 0.18 0.14
- added link mmwave_radar_link; visual cylinder length=0.09 radius=0.18
Joints:
- removed joint radar_joint
- added joint als_lidar_joint: type fixed, parent base_link, child als_lidar_link, origin xyz=0.15 0 1.72 rpy=0 0 0
- added joint gated_camera_joint: type fixed, parent base_link, child gated_camera_link, origin xyz=1.55 0 1.20 rpy=0 0 0
- added joint mmwave_radar_joint: type fixed, parent base_link, child mmwave_radar_link, origin xyz=-0.35 0 1.86 rpy=0 0 0

File: usv_ws/src/usv_description/urdf/wamv_base.urdf.xacro (robot description, xacro)
@@ -81,7 +81,11 @@
   <gazebo reference="base_link">
     <gravity>false</gravity>
+    <velocity_decay>
+      <linear>0.25</linear>
+      <angular>0.35</angular>
+    </velocity_decay>
     <material>Gazebo/Orange</material>
   </gazebo>
-  <link name="radar_link">
+  <link name="mmwave_radar_link">
     <visual>
       <origin xyz="0 0 0" rpy="0 0 0"/>
@@ -92,18 +96,18 @@
     </visual>
   </link>
-  <joint name="radar_joint" type="fixed">
-    <parent link="base_link"/>
-    <child link="radar_link"/>
+  <joint name="mmwave_radar_joint" type="fixed">
+    <parent link="base_link"/>
+    <child link="mmwave_radar_link"/>
     <origin xyz="-0.35 0 1.86" rpy="0 0 0"/>
   </joint>
-  <gazebo reference="radar_link">
-    <sensor type="ray" name="radar_sensor">
-      <pose>0 0 0 0 0 0</pose>
-      <visualize>true</visualize>
-      <update_rate>12</update_rate>
+  <gazebo reference="mmwave_radar_link">
+    <sensor type="ray" name="mmwave_radar_sensor">
+      <pose>0 0 0 0 0 0</pose>
+      <visualize>false</visualize>
+      <update_rate>8</update_rate>
       <ray>
         <scan>
           <horizontal>
-            <samples>720</samples>
+            <samples>360</samples>
             <resolution>1</resolution>
             <min_angle>-${pi}</min_angle>
@@ -122,10 +126,10 @@
         </noise>
       </ray>
-      <plugin name="gazebo_ros_radar" filename="libgazebo_ros_ray_sensor.so">
-        <ros>
-          <remapping>~/out:=radar/scan</remapping>
+      <plugin name="gazebo_ros_mmwave_radar" filename="libgazebo_ros_ray_sensor.so">
+        <ros>
+          <remapping>~/out:=mmwave_radar/scan</remapping>
         </ros>
         <output_type>sensor_msgs/LaserScan</output_type>
-        <frame_name>radar_link</frame_name>
+        <frame_name>mmwave_radar_link</frame_name>
       </plugin>
     </sensor>
@@ -147,11 +151,11 @@
     <sensor type="depth" name="depth_camera">
       <pose>0 0 0 0 0 0</pose>
-      <visualize>true</visualize>
-      <update_rate>30.0</update_rate>
+      <visualize>false</visualize>
+      <update_rate>10.0</update_rate>
       <camera>
         <horizontal_fov>1.3962634</horizontal_fov>
         <image>
-          <width>800</width>
-          <height>600</height>
+          <width>640</width>
+          <height>480</height>
           <format>R8G8B8</format>
         </image>
@@ -174,4 +178,98 @@
     </sensor>
   </gazebo>
+  <link name="gated_camera_link">
+    <visual>
+      <geometry>
+        <box size="0.20 0.18 0.14"/>
+      </geometry>
+      <material name="camera_blue"/>
+    </visual>
+  </link>
+  <joint name="gated_camera_joint" type="fixed">
+    <parent link="base_link"/>
+    <child link="gated_camera_link"/>
+    <origin xyz="1.55 0 1.20" rpy="0 0 0"/>
+  </joint>
+  <gazebo reference="gated_camera_link">
+    <sensor type="camera" name="gated_camera">
+      <pose>0 0 0 0 0 0</pose>
+      <visualize>true</visualize>
+      <update_rate>15.0</update_rate>
+      <camera>
+        <horizontal_fov>1.20</horizontal_fov>
+        <image>
+          <width>640</width>
+          <height>480</height>
+          <format>R8G8B8</format>
+        </image>
+        <clip>
+          <near>0.05</near>
+          <far>120.0</far>
+        </clip>
+      </camera>
+      <plugin name="gazebo_ros_gated_camera" filename="libgazebo_ros_camera.so">
+        <ros>
+          <remapping>~/image_raw:=gated_camera/image_raw</remapping>
+          <remapping>~/camera_info:=gated_camera/camera_info</remapping>
+        </ros>
+        <camera_name>gated_camera</camera_name>
+        <frame_name>gated_camera_link</frame_name>
+      </plugin>
+    </sensor>
+  </gazebo>
+  <link name="als_lidar_link">
+    <visual>
+      <origin xyz="0 0 0" rpy="0 0 0"/>
+      <geometry>
+        <cylinder radius="0.12" length="0.12"/>
+      </geometry>
+      <material name="sensor_black"/>
+    </visual>
+  </link>
+  <joint name="als_lidar_joint" type="fixed">
+    <parent link="base_link"/>
+    <child link="als_lidar_link"/>
+    <origin xyz="0.15 0 1.72" rpy="0 0 0"/>
+  </joint>
+  <gazebo reference="als_lidar_link">
+    <sensor type="ray" name="als_lidar">
+      <pose>0 0 0 0 0 0</pose>
+      <visualize>false</visualize>
+      <update_rate>5</update_rate>
+      <ray>
+        <scan>
+          <horizontal>
+            <samples>240</samples>
+            <resolution>1</resolution>
+            <min_angle>-${pi}</min_angle>
+            <max_angle>${pi}</max_angle>
+          </horizontal>
+          <vertical>
+            <samples>8</samples>
+            <resolution>1</resolution>
+            <min_angle>-0.28</min_angle>
+            <max_angle>0.12</max_angle>
+          </vertical>
+        </scan>
+        <range>
+          <min>0.3</min>
+          <max>90.0</max>
+          <resolution>0.03</resolution>
+        </range>
+        <noise>
+          <type>gaussian</type>
+          <mean>0.0</mean>
+          <stddev>0.015</stddev>
+        </noise>
+      </ray>
+      <plugin name="gazebo_ros_als_lidar" filename="libgazebo_ros_ray_sensor.so">
+        <ros>
+          <remapping>~/out:=als/points</remapping>
+        </ros>
+        <output_type>sensor_msgs/PointCloud2</output_type>
+        <frame_name>als_lidar_link</frame_name>
+      </plugin>
+    </sensor>
+  </gazebo>
   <link name="sonar_link">
     <visual>
@@ -191,6 +289,6 @@
     <sensor type="ray" name="sonar_sensor">
       <pose>0 0 0 0 0 0</pose>
-      <visualize>true</visualize>
-      <update_rate>8</update_rate>
+      <visualize>false</visualize>
+      <update_rate>6</update_rate>
       <ray>
         <scan>
@@ -210,9 +308,8 @@
       <plugin name="gazebo_ros_sonar" filename="libgazebo_ros_ray_sensor.so">
         <ros>
-          <remapping>~/out:=sonar/range</remapping>
-        </ros>
-        <output_type>sensor_msgs/Range</output_type>
+          <remapping>~/out:=sonar/scan</remapping>
+        </ros>
+        <output_type>sensor_msgs/LaserScan</output_type>
         <frame_name>sonar_link</frame_name>
-        <radiation_type>ultrasound</radiation_type>
       </plugin>
     </sensor>

Commit message: 简单的跟踪5.23

File: usv_ws/src/usv_description/urdf/wamv.urdf (robot description, URDF)
Before this commit: robot fog_usv, 7 links, 6 joints
Links:
- added link radar_10m_link; visual cylinder length=0.09 radius=0.18
- added link radar_1m_link; visual cylinder length=0.09 radius=0.18
- added link radar_1p5m_link; visual cylinder length=0.09 radius=0.18
- added link radar_1p9m_link; visual cylinder length=0.09 radius=0.18
- added link radar_4m_link; visual cylinder length=0.09 radius=0.18
Joints:
- added joint radar_10m_joint: type fixed, parent base_link, child radar_10m_link, origin xyz=-0.35 0 10.0 rpy=0 0 0
- added joint radar_1m_joint: type fixed, parent base_link, child radar_1m_link, origin xyz=-0.35 0 1.0 rpy=0 0 0
- added joint radar_1p5m_joint: type fixed, parent base_link, child radar_1p5m_link, origin xyz=-0.35 0 1.5 rpy=0 0 0
- added joint radar_1p9m_joint: type fixed, parent base_link, child radar_1p9m_link, origin xyz=-0.35 0 1.9 rpy=0 0 0
- added joint radar_4m_joint: type fixed, parent base_link, child radar_4m_link, origin xyz=-0.35 0 4.0 rpy=0 0 0

File: usv_ws/src/usv_description/urdf/wamv_base.urdf.xacro (robot description, xacro)
@@ -1,4 +1,5 @@
 <?xml version="1.0"?>
 <robot xmlns:xacro="http://www.ros.org/wiki/xacro" name="fog_usv">
+  <xacro:arg name="enable_c3_mmwave" default="true"/>
   <material name="pontoon_orange">
     <color rgba="1.0 0.42 0.08 1.0"/>
@@ -13,4 +14,54 @@
     <color rgba="0.08 0.22 0.34 1.0"/>
   </material>
+  <xacro:macro name="c3_raw_mmwave_sensor" params="name height topic">
+    <link name="${name}_link">
+      <visual>
+        <origin xyz="0 0 0" rpy="0 0 0"/>
+        <geometry>
+          <cylinder radius="0.18" length="0.09"/>
+        </geometry>
+        <material name="sensor_black"/>
+      </visual>
+    </link>
+    <joint name="${name}_joint" type="fixed">
+      <parent link="base_link"/>
+      <child link="${name}_link"/>
+      <origin xyz="-0.35 0 ${height}" rpy="0 0 0"/>
+    </joint>
+    <gazebo reference="${name}_link">
+      <sensor type="ray" name="${name}_raw_sensor">
+        <pose>0 0 0 0 0 0</pose>
+        <visualize>false</visualize>
+        <update_rate>15</update_rate>
+        <ray>
+          <scan>
+            <horizontal>
+              <samples>400</samples>
+              <resolution>1</resolution>
+              <min_angle>-1.0472</min_angle>
+              <max_angle>1.0472</max_angle>
+            </horizontal>
+          </scan>
+          <range>
+            <min>1.0</min>
+            <max>800.0</max>
+            <resolution>0.5</resolution>
+          </range>
+          <noise>
+            <type>gaussian</type>
+            <mean>0.0</mean>
+            <stddev>0.08</stddev>
+          </noise>
+        </ray>
+        <plugin name="gazebo_ros_${name}_raw" filename="libgazebo_ros_ray_sensor.so">
+          <ros>
+            <remapping>~/out:=${topic}</remapping>
+          </ros>
+          <output_type>sensor_msgs/LaserScan</output_type>
+          <frame_name>${name}_link</frame_name>
+        </plugin>
+      </sensor>
+    </gazebo>
+  </xacro:macro>
   <link name="base_footprint"/>
   <joint name="base_footprint_joint" type="fixed">
@@ -135,4 +186,11 @@
     </sensor>
   </gazebo>
+  <xacro:if value="$(arg enable_c3_mmwave)">
+    <xacro:c3_raw_mmwave_sensor name="radar_10m" height="10.0" topic="radar_10m/raw_scan"/>
+    <xacro:c3_raw_mmwave_sensor name="radar_4m" height="4.0" topic="radar_4m/raw_scan"/>
+    <xacro:c3_raw_mmwave_sensor name="radar_1p9m" height="1.9" topic="radar_1p9m/raw_scan"/>
+    <xacro:c3_raw_mmwave_sensor name="radar_1p5m" height="1.5" topic="radar_1p5m/raw_scan"/>
+    <xacro:c3_raw_mmwave_sensor name="radar_1m" height="1.0" topic="radar_1m/raw_scan"/>
+  </xacro:if>
   <link name="depth_camera_link">
     <visual>
